Commit message: 20211205

File: my_open_manipulator_description/urdf/open_manipulator_robot.urdf.xacro (robot description, xacro)
@@ -10,6 +10,42 @@
   <!-- Import URDF -->
   <xacro:include filename="$(find open_manipulator_description)/urdf/open_manipulator.urdf.xacro" />
+  <xacro:macro name="cylinder_inertia" params="m r h">
+        <inertia  ixx="${m*(3*r*r+h*h)/12}" ixy = "0" ixz = "0"
+                    iyy="${m*(3*r*r+h*h)/12}" iyz = "0"
+                    izz="${m*r*r/2}" />
+  </xacro:macro>
+  <xacro:macro name="box_inertia" params="m x y z">
+          <inertia  ixx="${m*(y*y+z*z)/12}" ixy = "0" ixz = "0"
+                    iyy="${m*(x*x+z*z)/12}" iyz = "0"
+                    izz="${m*(x*x+z*z)/12}" />
+  </xacro:macro>
+  <xacro:macro name="sphere_inertia" params="m r">
+          <inertia  ixx="${2*m*r*r/5}" ixy = "0" ixz = "0"
+                    iyy="${2*m*r*r/5}" iyz = "0"
+                    izz="${2*m*r*r/5}" />
+  </xacro:macro>
+  <material name="LightGrey">
+      <color rgba="0.7 0.7 0.7 1.0" />
+  </material>
   <!-- World -->
   <link name="world"/>
+  <link name="baseplate_link">
+    <visual>
+      <origin xyz="0.125 0 -0.004" />
+      <geometry>
+        <box size="0.3 0.3 0.008" />
+      </geometry>
+      <material name="LightGrey"/>
+    </visual>
+    <inertial>
+      <mass value="1"/>
+      <xacro:box_inertia m="1" x="0.3" y="0.3" z="0.008"/>
+    </inertial>
+  </link>
+  <joint name="baseplate_joint" type="fixed">
+    <origin xyz="0 0 0" />
+    <parent link="world" />
+    <child link="baseplate_link" />
+  </joint>
   <!-- World fixed joint-->
   <joint name="world_fixed" type="fixed">

Commit message: 20220114

File: my_open_manipulator_description/urdf/open_manipulator_robot.urdf.xacro (robot description, xacro)
@@ -54,3 +54,10 @@
     <child link="link1"/>
   </joint>
+  <!-- tool center point -->
+  <link name="tcp_link" />
+  <joint name="tool0_link" type="fixed">
+    <parent link="end_effector_link" />
+    <child link="tcp_link" />
+    <origin xyz="0.0 0.0 0.0" rpy="0.0 0.0 0.0"/>
+  </joint>
 </robot>
